File: Examples/COMET1_CCT_Board_WIP/COMET1_CCT.kicad_pcb (KiCad board)
At the start: 4 copper layers, 82 x 66 mm, 96 parts, among them J1 DF11-10DS-2DSA, J10 Molex_01x02, J11 Molex_01x02, J12 Molex_01x02, J13 Conn_02x03_Odd_Even, J2 DF11-10DS-2DSA, J3 Micro_SD_Card, J4 Pin_01x02, J5 USBC_Conn, J6 RJ45_LED_Shielded, J7 Molex_01x02, J8 Molex_01x02, J9 Molex_01x02, U1 RP2350_80QFN, U2 S25FL128, U3 NCP1117_3.3, U4 MAX490ESA+T, U5 LM27313XMFX_NOPB, U6 PAC1934T-I_JQ, U7 MCP96RL00-E_MX, U8 MCP96RL00-E_MX, U9 STS4L-AD1B-R3, X1 ABM8-272-T3

Commit message: Example files update
Parts:
- removed C20, C21: DNP, 0_Capacitors:C_0603_1608_DensityHigh
- removed C24: 100nF, 0_Capacitors:C_0603_1608_DensityHigh
- removed F2: Fuse, 0_Passives:Fuse_2512_6332Metric
- removed J6: RJ45_LED_Shielded, 0_Connectors:RJ45_56L-88112011
- removed the R13 at (118.4, 69.4)
- removed the R22 at (102.0, 98.5)
- removed U4: MAX490ESA+T, 0_Sensors:SOIC-8_3.9x4.9mm_P1.27mm
- added C34: 100nF, 0_Capacitors:C_0603_1608_DensityHigh, F.Cu at (129.9, 97.0)
- added J14: RJ45_LED_Shielded, 0_Connectors:RJ45_56L-88112011, F.Cu at (124.9, 80.9)
- added LED3: Red, 0_Passives:LED_0603_1608Metric, F.Cu at (169.3, 76.4)
- added Q1: MMBT5551, 0_Passives:SOT-23, F.Cu at (162.6, 113.7)
- added R17: 120R, 0_Resistors:R_0603_1608_DensityHigh, F.Cu at (123.5, 94.5)
- added R9: 1kR, 0_Resistors:R_0402_1005_DensityMedium, F.Cu at (161.6, 111.0)
- added U10: ISL83488, 0_Sensors:SOIC-8_3.9x4.9mm_P1.27mm, F.Cu at (128.6, 93.2)
- BUZ1: footprint 0_Passives:BUZZER,7.5x7.5mm -> 0_Passives:BUZZER,5x5mm
- C19: moved to F.Cu
- C22, C23, C29, C31: value 10nF -> 100nF
- D1: value ~ -> 1N4148WS; footprint 0_Passives:LED_0805_2012Metric -> 0_Passives:D_SOD-323
- D3: footprint 0_Passives:D_0805_2012Metric -> 0_Passives:D_SOD-123
- F1: footprint 0_Passives:Fuse_2512_6332Metric -> 0_Power:Fuse_1210_3225Metric
- J13: value Conn_02x03_Odd_Even -> Conn_02x03
- L1: value 1uH -> 3.3uH
- R1, R2: footprint 0_Resistors:R_0402_1005_DensityHigh -> 0_Resistors:R_0603_1608_DensityHigh
- R10: renamed from R9; value 4k7R -> 4.7kR
- R11: renamed from R10; value 4k7R -> 4.7kR
- R14: value 220R -> 51R; moved to F.Cu
- R16: value 120R -> 220R; moved to B.Cu
- R18: renamed from R17; value 0R2 -> 0.1R
- R19: renamed from R18; value 0R2 -> 0.1R
- R20: renamed from R19; value 0R2 -> 0.1R
- R21: renamed from R20; value 118kR -> 120kR; moved to F.Cu
- R22: renamed from R21; value 13.3kR -> 13kR; moved to F.Cu
- R5: footprint 0_Resistors:R_0603_1608_DensityHigh -> 0_Resistors:R_0402_1005_DensityMedium
- R6: footprint 0_Resistors:R_0402_1005_DensityHigh -> 0_Resistors:R_0402_1005_DensityMedium
- R7, R8: value ?220R? -> 51R
- U1: value RP2350_80QFN -> RP2350B
- U5: value LM27313XMFX_NOPB -> LM27313; footprint 0_Power:SOT95P280X145-5N -> 0_Power:SOT-23-5
- U6: value PAC1934T-I_JQ -> PAC1934; footprint 0_Sensors:QFN65P400X400X55-17N-D -> 0_Sensors:PAC1934T-I_JQ
- U7, U8: value MCP96RL00-E_MX -> MCP96R00; footprint 0_Sensors:QFN65P500X500X100-21N-D -> 0_Sensors:MCP9600L00
- U9: value STS4L-AD1B-R3 -> STS4L
- moved R14 102.9 mm to (170.9, 76.4), turned to 90 degrees
- moved R16 66.2 mm to (135.7, 84.6), turned to 180 degrees
- moved D1 63.0 mm to (168.7, 112.3), turned to 180 degrees
- moved BUZ1 61.7 mm to (168.7, 117.1), turned to 180 degrees
- moved C19 61.3 mm to (112.9, 113.3), turned to 180 degrees
- moved G*** 57.2 mm to (179.9, 105.8), turned to 90 degrees
- moved F1 56.6 mm to (169.5, 81.7)
- moved R2 56.0 mm to (145.5, 90.6)
- moved C10 55.8 mm to (152.0, 95.5)
- moved C14 55.8 mm to (152.5, 99.2)
- moved C16 55.8 mm to (143.1, 110.2)
- moved C17 55.8 mm to (146.1, 110.2)
- moved C18 55.8 mm to (147.4, 84.0)
- moved C2 55.8 mm to (147.5, 93.7)
- moved C26 55.8 mm to (179.8, 114.7)
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- renumbered R11 to R12, R12 to R13
Connections:
- net /CCT Board Schematic/USBC/CC1 renamed /CCT Board Schematic/Comms/CC1
- net /CCT Board Schematic/USBC/CC2 renamed /CCT Board Schematic/Comms/CC2
- net /CCT Board Schematic/USBC/D+ renamed /CCT Board Schematic/Comms/D+
- net /CCT Board Schematic/USBC/D- renamed /CCT Board Schematic/Comms/D-
- net /CCT Board Schematic/USBC/VBUS_PF renamed /CCT Board Schematic/Comms/VBUS_PF
- BUZ1 pad 1: /CCT Board Schematic/MCU & Peripherals/STATUS_BUZZER+ -> +3V3
- BUZ1 pad 2: /CCT Board Schematic/MCU & Peripherals/STATUS_BUZZER- -> Net-(BUZ1--)
- C22 pad 2: VBUS_F -> VBUS
- C23 pad 1: Net-(U3-VO) -> +3V3
- D1 pad 1: /CCT Board Schematic/MCU & Peripherals/STATUS_BUZZER+ -> +3V3
- D1 pad 2: /CCT Board Schematic/MCU & Peripherals/STATUS_BUZZER- -> Net-(BUZ1--)
- D2 pad 4: /CCT Board Schematic/USBC/USB_D+ -> /CCT Board Schematic/Comms/USB_D+
- D2 pad 6: /CCT Board Schematic/USBC/USB_D- -> /CCT Board Schematic/Comms/USB_D-
- J1 pad 1: /CCT Board Schematic/MCU & Peripherals/PYRO_SENSE -> /CCT Board Schematic/MCU & Peripherals/Servo3_PWM
- J1 pad 3: /CCT Board Schematic/MCU & Peripherals/PYRO_IN -> /CCT Board Schematic/MCU & Peripherals/Servo2_PWM
- J1 pad 5: /CCT Board Schematic/MCU & Peripherals/PYRO_SEN -> /CCT Board Schematic/MCU & Peripherals/Servo1_PWM
- J2 pad 10: GND -> /CCT Board Schematic/MCU & Peripherals/PYRO_IN
- J2 pad 3: /CCT Board Schematic/MCU & Peripherals/Servo1_PWM -> +3V3
- J2 pad 5: /CCT Board Schematic/MCU & Peripherals/Servo2_PWM -> GND
- J2 pad 6: GND -> /CCT Board Schematic/MCU & Peripherals/PYRO_ST2
- J2 pad 7: /CCT Board Schematic/MCU & Peripherals/Servo3_PWM -> GND
- J2 pad 8: GND -> /CCT Board Schematic/MCU & Peripherals/PYRO_ST1
- R1 pad 1: /CCT Board Schematic/MCU & Peripherals/USB_D+ -> /CCT Board Schematic/Comms/USB_D+
- R14 pad 1: Net-(J6-Pad10) -> GND
- R14 pad 2: GND -> Net-(LED3-K)
- R15 pad 1: GND -> Net-(J14-Pad10)
- R15 pad 2: Net-(J6-Pad12) -> GND
- R16 pad 1: /CCT Board Schematic/RS485/RS485_RX+ -> GND
- R16 pad 2: /CCT Board Schematic/RS485/RS485_RX- -> Net-(J14-Pad12)
- R2 pad 1: /CCT Board Schematic/MCU & Peripherals/USB_D- -> /CCT Board Schematic/Comms/USB_D-
- U1 pad 1: /CCT Board Schematic/MCU & Peripherals/FIRE_SIGNAL -> /CCT Board Schematic/Comms/FIRE_SIGNAL
- U1 pad 11: /CCT Board Schematic/MCU & Peripherals/Servo2_PWM -> /CCT Board Schematic/MCU & Peripherals/PYRO_ST1
- U1 pad 12: /CCT Board Schematic/MCU & Peripherals/SD_DAT1 -> /CCT Board Schematic/MCU & Peripherals/PYRO_IN
- U1 pad 13: /CCT Board Schematic/MCU & Peripherals/Servo3_PWM -> /CCT Board Schematic/MCU & Peripherals/SD_DAT1
- U1 pad 2: /CCT Board Schematic/MCU & Peripherals/ARM_SIGNAL -> /CCT Board Schematic/Comms/ARM_SIGNAL
- U1 pad 3: /CCT Board Schematic/MCU & Peripherals/FILL_SIGNAL -> /CCT Board Schematic/Comms/FILL_SIGNAL
- U1 pad 4: /CCT Board Schematic/MCU & Peripherals/RJ45_LED2 -> /CCT Board Schematic/Comms/RJ45_LED2
- U1 pad 44: /CCT Board Schematic/MCU & Peripherals/STATUS_BUZZER- -> unconnected-(U1A-GPIO35-Pad44)
- U1 pad 45: /CCT Board Schematic/MCU & Peripherals/STATUS_BUZZER+ -> /CCT Board Schematic/MCU & Peripherals/STATUS_BUZZER
- U1 pad 53: unconnected-(U1A-GPIO42_ADC2-Pad53) -> /CCT Board Schematic/MCU & Peripherals/Servo3_PWM
- U1 pad 54: /CCT Board Schematic/MCU & Peripherals/PYRO_SENSE -> unconnected-(U1A-GPIO43_ADC3-Pad54)
- U1 pad 55: /CCT Board Schematic/MCU & Peripherals/PYRO_IN -> /CCT Board Schematic/MCU & Peripherals/Servo2_PWM
- U1 pad 56: /CCT Board Schematic/MCU & Peripherals/PYRO_SEN -> unconnected-(U1A-GPIO45_ADC5-Pad56)
- U1 pad 57: unconnected-(U1A-GPIO46_ADC6-Pad57) -> /CCT Board Schematic/MCU & Peripherals/Servo1_PWM
- U1 pad 6: /CCT Board Schematic/MCU & Peripherals/RS485_TX -> /CCT Board Schematic/Comms/RS485_TX
- U1 pad 7: /CCT Board Schematic/MCU & Peripherals/RS485_RX -> /CCT Board Schematic/Comms/RS485_RX
- U1 pad 8: /CCT Board Schematic/MCU & Peripherals/RJ45_LED1 -> /CCT Board Schematic/Comms/RJ45_LED1
- U1 pad 9: /CCT Board Schematic/MCU & Peripherals/Servo1_PWM -> /CCT Board Schematic/MCU & Peripherals/PYRO_ST2
- U3 pad 2: Net-(U3-VO) -> +3V3
- U3 pad 3: VBUS_F -> VBUS
- U6 pad 6: Net-(U6-ADDRSEL) -> GND
Routing:
- net (no net): track 97.7 -> 0.00 mm, vias 2 -> 0
- net /CCT Board Schematic/MCU & Peripherals/STATUS_BUZZER-: track 23.8 -> 0.00 mm
- net /CCT Board Schematic/Comms/RJ45_LED1: track 0.00 -> 22.8 mm, vias 0 -> 1
- net +3V3: track 64.3 -> 86.2 mm, vias 16 -> 25
- net /CCT Board Schematic/MCU & Peripherals/FILL_SIGNAL: track 21.7 -> 0.00 mm
- net /CCT Board Schematic/MCU & Peripherals/PYRO_SENSE: track 21.4 -> 0.00 mm
- net /CCT Board Schematic/MCU & Peripherals/STATUS_BUZZER+: track 20.8 -> 0.00 mm
- net /CCT Board Schematic/Comms/FILL_SIGNAL: track 0.00 -> 20.7 mm
- net /CCT Board Schematic/RS485/RS485_RX-: track 20.5 -> 0.00 mm
- net /CCT Board Schematic/MCU & Peripherals/PYRO_SEN: track 20.1 -> 0.00 mm
- net /CCT Board Schematic/RS485/RS485_RX+: track 19.5 -> 0.00 mm
- net /CCT Board Schematic/Comms/RS485_RX-: track 0.00 -> 19.5 mm
- net /CCT Board Schematic/MCU & Peripherals/ARM_SIGNAL: track 19.0 -> 0.00 mm
- net /CCT Board Schematic/Comms/USB_D-: track 0.00 -> 18.8 mm
- net /CCT Board Schematic/Comms/RS485_RX+: track 0.00 -> 18.4 mm
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- removed copper zone on F.Cu, net Net-(U3-VO)
Other:
- rule pad_to_mask_clearance: 0.1 -> 0.05
- board text added: "3v3"
- board text added: "Board - Board Connector 1"
- board text added: "Board - Board Connector 2"
- board text added: "Board Dimensions (Scale 1:1 @ A4)"
- board text added: "Hole - Ø 3.2mm M3 Pad - Ø 6.4mm"
- board text added: "I2C"
- board text added: "J1"
- board text added: "J2"
- board text added: "PCB: V1 01/26 FIRMWARE:"
- board text added: "PressureA"
- board text added: "PressureB"
- board text added: "PressureC"
- board text added: "RJ45"
- board text added: "SCL"
- board text added: "SDA"
- board text added: "ThermoA"
- board text added: "ThermoB"
- board text added: "USB C"
- board text added: "ew8g21"
- board text added: "uSD Card"
- board text removed: "??? ??? ???"
- board text removed: "??? ??? ??? ??? ??? (slot) ??? ??? ??? ??? ???"
- board text removed: "???mm"
- board text removed: "???mm (?oz)"
- board text removed: "???mm ???mm ???mm ???mm ???mm ???mm ???mm ???mm ???mm ???mm"
- board text removed: "ASSEMBLY NOTES (UNLESS OTHERWISE SPECIFIED) 1) DO NOT POPULATE PARTS ARE MARKED WITH A RED CROSS. 2) DO NOT POPULATE PARTS ARE NOT PRESENT IN THE BOM. 3) IF CONFLICTING INFORMATION IS FOUND BETWEEN THE ASSEMBLY FILE AND BOM, BOM SHOULD BE USED AS THE MAIN SOURCE."
- board text removed: "All dimensions are in millimeters unless otherwise specified."
- board text removed: "B.Mask"
- board text removed: "B.Paste"
- board text removed: "B.Silkscreen"
- board text removed: "Back Side"
- board text removed: "Bottom Assembly (Scale 1:1)"
- board text removed: "Bottom Fabrication (Scale 1:1)"
- board text removed: "Bottom Test Points (Scale 1:1)"
- board text removed: "Components"
- board text removed: "Copper"
- board text removed: "Core"
- board text removed: "Count"
- board text removed: "Dielectric"
- board text removed: "Dielectric Material"
- board text removed: "Drill Drawing (Top View) (Scale 1:1)"
- board text removed: "F.Mask"
- board text removed: "F.Paste"
- board text removed: "F.Silkscreen"
- board text removed: "FABRICATION NOTES (UNLESS OTHERWISE SPECIFIED) 1) OUTLINE DEFINED IN SEPARATE GERBER FILE WITH {dblquote}Edge_Cuts.GBR{dblquote} SUFFIX. DIMENSIONS OF CIRCUMSIZED RECTANGLE SHOWN ON THIS DWG FOR REF ONLY. 2) SEE SEPARATE DRILL FILES WITH {dblquote}.DRL{dblquote} SUFFIX FOR HOLE LOCATIONS. SELECTED HOLE LOCATIONS SHOWN ON THIS DWG FOR REF ONLY. 3) IMPEDANCE CONTROL REQUIRED. Microstrip 100-Ohm Dif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"
- board text removed: "FR-4"
- board text removed: "Front Side"
- board text removed: "GBR"
- board text removed: "Gerber"
- board text removed: "Hole Size"
- board text removed: "Internal Plane"
- board text removed: "L1 (Sig, PWR)"
- board text removed: "L2 (GND)"
- board text removed: "L3 (Sig, PWR)"
- board text removed: "L4 (Sig, PWR)"
- board text removed: "L5 (GND)"
- board text removed: "L6 (Sig, PWR)"
- board text removed: "Layer"
- board text removed: "Layer Stack Legend"
- board text removed: "Legend"
- board text removed: "Material"
- board text removed: "Net"
- board text removed: "Note: external layer thicknesses are specified after plating."
- board text removed: "PCB3D_BR_BOARDNAME"
- board text removed: "PCB3D_TL_BOARDNAME"
- board text removed: "Paste Mask"
- board text removed: "Plated"
- board text removed: "Plated Plated Plated Plated Plated Plated Plated Plated Plated Unplated"
- board text removed: "Prepreg"
- board text removed: "Ref."
- board text removed: "Signal"
- board text removed: "Solder Mask"
- board text removed: "Solder Resist"
- board text removed: "Symbol"
- board text removed: "THT SMD Total"
- board text removed: "TP? TP? TP?"
- board text removed: "Thickness"
- board text removed: "Top Assembly (Scale 1:1)"
- board text removed: "Top Fabrication (Scale 1:1)"
- board text removed: "Top Test Points (Scale 1:1)"
- board text removed: "Total"
- board text removed: "Total thickness: 1.62mm"
- board text removed: "Type"
- board text removed: "X"
- board text removed: "X [mm]"
- board text removed: "Y"
- board text removed: "Y [mm]"
- board text removed: "ew8g21 12/25"
