File: Examples/COMET1_CCT_Board_WIP/COMET1_CCT.kicad_sch (KiCad schematic)
At the start: 0 parts

Commit message: Example files update
Other:
- sheet Block Diagram: file Block Diagram.kicad_sch -> SubSchematics/Block Diagram.kicad_sch
- sheet CCT Board Schematic: file CCT Board Schematic.kicad_sch -> SubSchematics/CCT Board Schematic.kicad_sch
- note added: "ADD FUNCTIONALITY FOR EXTERNAL WARNING LIGHT AT ROCKET FOR ARMING AND COUNTDOWN PCB STITCHING VIAS PCB VCUTS/PANEL? + TOOLING HOLES"
- note added: "CCT Board Schematic"
- note added: "MCU & Peripherals"
- note added: "RS485"
- note added: "Sensors"
- note added: "USBC"
- note removed: "Power - Sequencing"
- note removed: "Project Architecture"
- note removed: "Random Sheet 1"
- note removed: "Random Sheet 2"
- note removed: "Revision History"
