File: Examples/COMET1_CCT_Board_WIP/SubSchematics/MCU & Peripherals.kicad_sch (KiCad schematic)
At the start: 41 parts, among them J12 Molex_01x02, J13 Conn_02x03_Odd_Even, J3 Micro_SD_Card, J4 Pin_01x02, U1 RP2350_80QFN, U2 S25FL128, X1 ABM8-272-T3

Commit message: Example files update
Parts:
- added Q1: MMBT5551, 0_Passives:SOT-23, symbol 0_Passives:MMBT5551
- added R9: 1kR, 0_Resistors:R_0402_1005_DensityMedium, symbol 0_Passives:R
- BUZ1: footprint 0_Passives:BUZZER,7.5x7.5mm -> 0_Passives:BUZZER,5x5mm; MPN (none) -> KSSG33J12Y; Min Qty (none) -> 5; Order Code (none) -> 4245943; Part Link (none) -> https://uk.farnell.com/kingstate/kssg33j12y/magnetic-transd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; Price Per (none) -> 1.06; Supplier (none) -> Farnell
- C1, C15, C2, C3: MPN (none) -> CL05A475MP5NRNC; Min Qty (none) -> 20; Order Code (none) -> C23733; Price Per (none) -> 0.0035; Supplier (none) -> JLCPCB
- C10, C11, C12, C13, C14, C4, C5, C6, C7, C8, C9: MPN (none) -> CL05B104KO5NNNC; Min Qty (none) -> 20; Order Code (none) -> C1525; Price Per (none) -> 0.0009; Supplier (none) -> JLCPCB
- C16, C17: MPN (none) -> 0402CG150J500NT; Min Qty (none) -> 20; Order Code (none) -> C1548; Price Per (none) -> 0.0007; Supplier (none) -> JLCPCB
- C18, C19: MPN (none) -> CC0603KRX7R9BB104; Min Qty (none) -> 20; Order Code (none) -> C14663; Price Per (none) -> 0.002; Supplier (none) -> JLCPCB
- D1: value ~ -> 1N4148WS; footprint 0_Passives:LED_0805_2012Metric -> 0_Passives:D_SOD-323; MPN (none) -> 1N4148WS; Min Qty (none) -> 20; Order Code (none) -> C2128; Price Per (none) -> 0.0062; Supplier (none) -> JLCPCB
- J12: Min Qty (none) -> 1; Order Code (none) -> 3103081; Part Link (none) -> https://uk.farnell.com/molex/502352-0201/wtb-conn-header-2p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; Price Per (none) -> 0.95; Supplier (none) -> Farnell; Supplier Link https://uk.farnell.com/molex/502352-0201/wtb-conn-header-2p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 -> (none)
- J13: value Conn_02x03_Odd_Even -> Conn_02x03; symbol Connector_Generic:Conn_02x03_Odd_Even -> 0_Connectors:Conn_02x03_Odd_Even; MPN (none) -> N/A
- J3: MPN (none) -> 47219-2001; Min Qty (none) -> 1; Order Code (none) -> 2614940; Part Link (none) -> https://uk.farnell.com/molex/47219-2001/connector-micro-sd-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; Price Per (none) -> 1.87; Supplier (none) -> Farnell
- J4: MPN (none) -> N/A
- L1: value 1uH -> 3.3uH; MPN (none) -> AOTA-B201610S3R3-101-T; Min Qty (none) -> 5; Order Code (none) -> C42411119; Price Per (none) -> 0.14; Supplier (none) -> JLCPCB
- LED1: MPN (none) -> MP008288; Min Qty (none) -> 5; Order Code (none) -> 3796319; Part Link (none) -> https://uk.farnell.com/multicomp-pro/mp008288/led-green-90m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; Price Per (none) -> 0.13; Supplier (none) -> Farnell
- LED2: MPN (none) -> MP008277; Min Qty (none) -> 5; Order Code (none) -> 3796306; Part Link (none) -> https://uk.farnell.com/multicomp-pro/mp008277/led-red-220mc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; Price Per (none) -> 0.13; Supplier (none) -> Farnell
- R1, R2: footprint 0_Resistors:R_0402_1005_DensityHigh -> 0_Resistors:R_0603_1608_DensityHigh; MPN (none) -> 0603WAF270JT5E; Min Qty (none) -> 20; Order Code (none) -> C25190; Price Per (none) -> 0.0008; Supplier (none) -> JLCPCB
- R10: renamed from R9; value 4k7R -> 4.7kR; MPN (none) -> 0603WAF4701T5E; Min Qty (none) -> 20; Order Code (none) -> C23162; Price Per (none) -> 0.0008; Supplier (none) -> JLCPCB
- R11: renamed from R10; value 4k7R -> 4.7kR; MPN (none) -> 0603WAF4701T5E; Min Qty (none) -> 20; Order Code (none) -> C23162; Price Per (none) -> 0.0008; Supplier (none) -> JLCPCB
- R3: MPN (none) -> 0402WGF330JTCE; Min Qty (none) -> 20; Order Code (none) -> C25105; Price Per (none) -> 0.0004; Supplier (none) -> JLCPCB
- R4: MPN (none) -> 0603WAF1002T5E; Min Qty (none) -> 20; Order Code (none) -> C25804; Price Per (none) -> 0.0007; Supplier (none) -> JLCPCB
- R5: footprint 0_Resistors:R_0603_1608_DensityHigh -> 0_Resistors:R_0402_1005_DensityMedium; MPN (none) -> 0402WGF1001TCE; Min Qty (none) -> 20; Order Code (none) -> C11702; Price Per (none) -> 0.0004; Supplier (none) -> JLCPCB
- R6: footprint 0_Resistors:R_0402_1005_DensityHigh -> 0_Resistors:R_0402_1005_DensityMedium; MPN (none) -> 0402WGF1001TCE; Min Qty (none) -> 20; Order Code (none) -> C11702; Price Per (none) -> 0.0004; Supplier (none) -> JLCPCB
- R7, R8: value ?220R? -> 51R; MPN (none) -> 0603WAF510JT5E; Min Qty (none) -> 20; Order Code (none) -> C23197; Price Per (none) -> 0.0008; Supplier (none) -> JLCPCB
- U1: value RP2350_80QFN -> RP2350B; MPN (none) -> RP2350B; Min Qty (none) -> 1; Order Code (none) -> C42415655; Price Per (none) -> 0.89; Supplier (none) -> JLCPCB
- U2: Min Qty (none) -> 1; Order Code (none) -> 4128033; Part Link (none) -> https://uk.farnell.com/infineon/s25fl128lagmfi013/flash-mem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; Price Per (none) -> 1.62; Supplier (none) -> Farnell; Supplier Link https://uk.farnell.com/infineon/s25fl128lagmfi013/flash-mem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 -> (none)
- X1: MPN (none) -> ABM8-272-T3; Min Qty (none) -> 1; Order Code (none) -> 4331750; Part Link (none) -> https://uk.farnell.com/abracon/abm8-272-t3/crystal-12mhz-10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; Price Per (none) -> 0.67; Supplier (none) -> Farnell
Connections:
- net +3V3: now also BUZ1.1 (+), D1.1 (K)
- net GND: now also Q1.2 (E); no longer BUZ1.3 (GND)
- net PYRO_IN: now also U1.12 (GPIO13); no longer U1.55 (GPIO44_ADC4)
- net SD_DAT1: now also U1.13 (GPIO14); no longer U1.12 (GPIO13)
- net Servo1_PWM: now also U1.57 (GPIO46_ADC6); no longer U1.9 (GPIO11)
- net Servo2_PWM: now also U1.55 (GPIO44_ADC4); no longer U1.11 (GPIO12)
- net Servo3_PWM: now also U1.53 (GPIO42_ADC2); no longer U1.13 (GPIO14)
- net PYRO_SEN: no longer names the net of U1.56 (GPIO45_ADC5)
- net PYRO_SENSE: no longer names the net of U1.54 (GPIO43_ADC3)
- removed net STATUS_BUZZER+: BUZ1.1 (+), D1.1 (K), U1.45 (GPIO36)
- net STATUS_BUZZER-: no longer names the net of BUZ1.2 (-), D1.2 (A)
- net STATUS_BUZZER-: now also Q1.3 (C); no longer U1.44 (GPIO35)
- new net: Q1.1 (B), R9.2
- new net PYRO_ST1: U1.11 (GPIO12)
- new net PYRO_ST2: U1.9 (GPIO11)
- new net STATUS_BUZZER: R9.1, U1.45 (GPIO36)
- no-connect marks 21 -> 22
Other:
- note removed: "1v1 VDD Decoupling"
- note removed: "3v3 VDD Decoupling All 100nF"
- note removed: "4.7uF below VREG"
- note removed: "I2C Pull Ups"
- note removed: "Jumper to program with USB"
- title: Sheet Title A -> MCU & Peripherals
- moved on the sheet: C1, C10, C11, C12, C13, C14, C15, C16, C17, C18, C19, C2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
