File: Examples/COMET1_CCT_Board_WIP/SubSchematics/Sensors.kicad_sch (KiCad schematic)
At the start: 27 parts, among them J10 Molex_01x02, J11 Molex_01x02, J7 Molex_01x02, J8 Molex_01x02, J9 Molex_01x02, U5 LM27313XMFX_NOPB, U6 PAC1934T-I_JQ, U7 MCP96RL00-E_MX, U8 MCP96RL00-E_MX, U9 STS4L-AD1B-R3

Commit message: Example files update
Parts:
- removed R22: 0R, 0_Resistors:R_0805_2012_DensityHigh, symbol 0_Passives:R
- C25, C26: MPN (none) -> CL10A475KO8NNNC; Min Qty (none) -> 20; Order Code (none) -> C19666; Price Per (none) -> 0.007; Supplier (none) -> JLCPCB
- C27, C28, C30, C32, C33: MPN (none) -> CC0603KRX7R9BB104; Min Qty (none) -> 20; Order Code (none) -> C14663; Price Per (none) -> 0.002; Supplier (none) -> JLCPCB
- C29, C31: value 10nF -> 100nF; MPN (none) -> CC0603KRX7R9BB104; Min Qty (none) -> 20; Order Code (none) -> C14663; Price Per (none) -> 0.002; Supplier (none) -> JLCPCB
- D3: footprint 0_Passives:D_0805_2012Metric -> 0_Passives:D_SOD-123; MPN (none) -> B5819W SL; Min Qty (none) -> 20; Order Code (none) -> C8598; Price Per (none) -> 0.017; Supplier (none) -> JLCPCB
- J10, J11, J7, J8, J9: Min Qty (none) -> 1; Order Code (none) -> 3103081; Part Link (none) -> https://uk.farnell.com/molex/502352-0201/wtb-conn-header-2p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; Price Per (none) -> 0.95; Supplier (none) -> Farnell; Supplier Link https://uk.farnell.com/molex/502352-0201/wtb-conn-header-2p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 -> (none)
- L2: MPN (none) -> MCSD54-120MU; Min Qty (none) -> 1; Order Code (none) -> 1864116; Part Link (none) -> https://uk.farnell.com/multicomp-pro/mcsd54-120mu/inductor-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; Price Per (none) -> 0.25; Supplier (none) -> Farnell
- R18: renamed from R17; value 0R2 -> 0.1R; MPN (none) -> 1206W4F100LT5E; Min Qty (none) -> 15; Order Code (none) -> C25334; Price Per (none) -> 0.0037; Supplier (none) -> JLCPCB
- R19: renamed from R18; value 0R2 -> 0.1R; MPN (none) -> 1206W4F100LT5E; Min Qty (none) -> 15; Order Code (none) -> C25334; Price Per (none) -> 0.0037; Supplier (none) -> JLCPCB
- R20: renamed from R19; value 0R2 -> 0.1R; MPN (none) -> 1206W4F100LT5E; Min Qty (none) -> 15; Order Code (none) -> C25334; Price Per (none) -> 0.0037; Supplier (none) -> JLCPCB
- R21: renamed from R20; value 118kR -> 120kR; MPN (none) -> 0603WAF1203T5E; Min Qty (none) -> 20; Order Code (none) -> C25808; Price Per (none) -> 0.0008; Supplier (none) -> JLCPCB
- R22: renamed from R21; value 13.3kR -> 13kR; MPN (none) -> 0603WAF1302T5E; Min Qty (none) -> 20; Order Code (none) -> C22797; Price Per (none) -> 0.0008; Supplier (none) -> JLCPCB
- U5: value LM27313XMFX_NOPB -> LM27313; footprint 0_Power:SOT95P280X145-5N -> 0_Power:SOT-23-5; Min Qty (none) -> 1; Order Code (none) -> 3121547; Part Link (none) -> https://uk.farnell.com/texas-instruments/lm27313xmfx-nopb/d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; Price Per (none) -> 1.85; Supplier (none) -> Farnell; Supplier Link https://uk.farnell.com/texas-instruments/lm27313xmfx-nopb/d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 -> (none)
- U6: value PAC1934T-I_JQ -> PAC1934; footprint 0_Sensors:QFN65P400X400X55-17N-D -> 0_Sensors:PAC1934T-I_JQ; Height 0.55 -> (none); MPN (none) -> PAC1934T-I/JQ; Manufacturer_Name Microchip -> (none); Manufacturer_Part_Number PAC1934T-I/JQ -> (none); Min Qty (none) -> 1; Order Code (none) -> 2907898; Part Link (none) -> https://uk.farnell.com/microchip/pac1934t-i-jq/dc-power-ene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; Price Per (none) -> 1.72; Supplier (none) -> Farnell
- U7, U8: value MCP96RL00-E_MX -> MCP96R00; footprint 0_Sensors:QFN65P500X500X100-21N-D -> 0_Sensors:MCP9600L00; Height 1 -> (none); Manufacturer_Name Microchip -> (none); Manufacturer_Part_Number MCP96RL00-E/MX -> (none); Min Qty (none) -> 1; Order Code (none) -> 2991624; Part Link (none) -> https://uk.farnell.com/microchip/mcp96rl00-e-mx/thermocoupl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; Price Per (none) -> 3.49; Supplier (none) -> Farnell; Supplier Link https://uk.farnell.com/microchip/mcp96rl00-e-mx/thermocoupl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 -> (none)
- U9: value STS4L-AD1B-R3 -> STS4L; Min Qty (none) -> 1; Order Code (none) -> 4551122; Part Link (none) -> https://uk.farnell.com/sensirion/sts4l-ad1b-r3/temperature-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; Price Per (none) -> 0.52; Supplier (none) -> Farnell; Supplier Link https://uk.farnell.com/sensirion/sts4l-ad1b-r3/temperature-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 -> (none)
Connections:
- net GND: now also U6.6 (ADDRSEL)
Other:
- note added: "I2C - 0x20"
- note added: "I2C - 0x44"
- note added: "I2C - 0x60"
- note added: "I2C - 0x6E"
- note removed: "I2C Address: 0x40"
- note removed: "Potential I2C Addresses: 0x44, 0x45, 0x46"
- title: Sheet Title A -> Sensors
- moved on the sheet: C30, C32
