File: Examples/COMET1_PWR_Board_WIP/COMET1_PWR_Board.kicad_pcb (KiCad board)
At the start: 2 copper layers, 82 x 66 mm, 42 parts, among them J1 XT30_THT_H, J2 Molex_Block_01x02, J3 502352-0301, J4 502352-0301, J5 502352-0301, J6 DF11-10DP-2DSA, J7 DF11-10DP-2DSA, U1 NCP1117_3.3, U2 BV1HJ180EFJ-C, U3 MIC29302AWD, U4 MIC29302AWD

Commit message: Example files update
Parts:
- R5: value 4k7R -> 4.7kR
- moved J3 0.70 mm to (129.5, 131.8)
- moved J4 0.70 mm to (147.5, 131.8)
- moved J5 0.70 mm to (165.5, 131.8)
- moved C2 0.70 mm to (151.9, 102.0)
- moved C6 0.70 mm to (131.6, 117.0)
- moved FID2 0.70 mm to (166.5, 83.0)
- moved G*** 0.70 mm to (131.5, 88.0)
- moved J1 0.70 mm to (174.5, 88.0)
- moved LED1 0.70 mm to (151.5, 75.0)
- moved MH3 0.70 mm to (183.5, 77.0)
- moved R3 0.70 mm to (147.7, 75.0)
- moved R6 0.70 mm to (134.7, 122.5)
- moved R7 0.70 mm to (137.7, 122.5)
- moved R8 0.70 mm to (150.7, 122.5)
- moved R9 0.70 mm to (153.7, 122.5)
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Routing:
- net GND: vias 219 -> 215
Other:
- board text added: "Board - Board Connector 1"
- board text added: "Board - Board Connector 2"
- board text added: "Board Dimensions (Scale 1:1 @ A4)"
- board text added: "Hole - Ø 3.2mm M3 Pad - Ø 6.4mm"
- board text removed: "BOARD CONN. 1"
- board text removed: "BOARD CONN. 2"
- board text removed: "M3 Ø 3.2mm"
