File: CanSat_SensorSuite/Block Diagram.kicad_sch (KiCad schematic)
At the start: 0 parts

Commit message: Minor schematic adjustments
Other:
- note removed: "+??V"
- note removed: "+A3V3"
- company: ${COMPANY} -> (none)
- title: Block Diagram -> (none)
