File: CanSat_SensorSuite/SubSchematics/MCU & Peripherals.kicad_sch (KiCad schematic)
At the start: 41 parts, among them J1 Pin_01x02, J12 Molex_01x02, J13 Conn_02x03_Odd_Even, J3 Micro_SD_Card, U1 RP2350_80QFN, U2 S25FL128, X1 ABM8-272-T3

Commit message: Minor schematic changes
Parts:
- BUZ?: renamed from BUZ1; JLC Part Number (none) -> C95299; JLC Price (none) -> 0.17; MPN (none) -> MLT-7525
- C?: renamed from C16; JLC Part Number (none) -> C1548; JLC Price (none) -> 0.0007; MPN (none) -> 0402CG150J500NT
- C?: renamed from C7; JLC Part Number (none) -> C1525; JLC Price (none) -> 0.0009; MPN (none) -> CL05B104KO5NNNC
- C?: renamed from C10; JLC Part Number (none) -> C1525; JLC Price (none) -> 0.0009; MPN (none) -> CL05B104KO5NNNC
- C?: renamed from C13; JLC Part Number (none) -> C1525; JLC Price (none) -> 0.0009; MPN (none) -> CL05B104KO5NNNC
- C?: renamed from C14; JLC Part Number (none) -> C1525; JLC Price (none) -> 0.0009; MPN (none) -> CL05B104KO5NNNC
- C?: renamed from C3; JLC Part Number (none) -> C23733; JLC Price (none) -> 0.0035; MPN (none) -> CL05A475MP5NRNC
- C?: renamed from C6; JLC Part Number (none) -> C1525; JLC Price (none) -> 0.0009; MPN (none) -> CL05B104KO5NNNC
- C?: renamed from C2; JLC Part Number (none) -> C23733; JLC Price (none) -> 0.0035; MPN (none) -> CL05A475MP5NRNC
- C?: renamed from C15; JLC Part Number (none) -> C23733; JLC Price (none) -> 0.0035; MPN (none) -> CL05A475MP5NRNC
- C?: renamed from C1; JLC Part Number (none) -> C23733; JLC Price (none) -> 0.0035; MPN (none) -> CL05A475MP5NRNC
- C?: renamed from C8; JLC Part Number (none) -> C1525; JLC Price (none) -> 0.0009; MPN (none) -> CL05B104KO5NNNC
- C?: renamed from C5; JLC Part Number (none) -> C1525; JLC Price (none) -> 0.0009; MPN (none) -> CL05B104KO5NNNC
- C?: renamed from C9; JLC Part Number (none) -> C1525; JLC Price (none) -> 0.0009; MPN (none) -> CL05B104KO5NNNC
- C?: renamed from C4; JLC Part Number (none) -> C1525; JLC Price (none) -> 0.0009; MPN (none) -> CL05B104KO5NNNC
- C?: renamed from C18; JLC Part Number (none) -> C14663; JLC Price (none) -> 0.002; MPN (none) -> CC0603KRX7R9BB104
- C?: renamed from C19; JLC Part Number (none) -> C14663; JLC Price (none) -> 0.002; MPN (none) -> CC0603KRX7R9BB104
- C?: renamed from C11; JLC Part Number (none) -> C1525; JLC Price (none) -> 0.0009; MPN (none) -> CL05B104KO5NNNC
- C?: renamed from C17; JLC Part Number (none) -> C1548; JLC Price (none) -> 0.0007; MPN (none) -> 0402CG150J500NT
- C?: renamed from C12; JLC Part Number (none) -> C1525; JLC Price (none) -> 0.0009; MPN (none) -> CL05B104KO5NNNC
- D?: renamed from D1; footprint 0_Passives:LED_0805_2012Metric -> 0_Passives:D_SOD-323; JLC Part Number (none) -> C2128; JLC Price (none) -> 0.0064; MPN (none) -> 1N4148WS
- J?: renamed from J13; value Conn_02x03_Odd_Even -> Conn_02x03; JLC Part Number (none) -> N/A; JLC Price (none) -> N/A; MPN (none) -> N/A; now not fitted
- J?: renamed from J1; JLC Part Number (none) -> N/A; JLC Price (none) -> N/A; MPN (none) -> N/A; now not fitted
- J?: renamed from J3; Farnell Link (none) -> https://uk.farnell.com/molex/47219-2001/connector-micro-sd-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; Farnell Part Number (none) -> 2614940; Farnell Price (none) -> 1.87; JLC Part Number (none) -> C164170; JLC Price (none) -> 0.43; MPN (none) -> 47219-2001
- J?: renamed from J12; Farnell Link (none) -> https://uk.farnell.com/molex/502352-0201/wtb-conn-header-2p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; Farnell Part Number (none) -> 3103081; Farnell Price (none) -> 0.95; JLC Part Number (none) -> C587898; JLC Price (none) -> 0.22; Supplier Link https://uk.farnell.com/molex/502352-0201/wtb-conn-header-2p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 -> (none)
- L?: renamed from L1; value 1uH -> 3.3uH; Farnell Link (none) -> https://uk.farnell.com/abracon/aota-b201610s3r3-101-t/power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; Farnell Part Number (none) -> 4568814; Farnell Price (none) -> 1.4; JLC Part Number (none) -> C42411119; JLC Price (none) -> 0.14; MPN (none) -> AOTA-B201610S3R3-101-T
- LED?: renamed from LED1; JLC Part Number (none) -> C12624; JLC Price (none) -> 0.009; MPN (none) -> KT-0603G
- LED?: renamed from LED2; JLC Part Number (none) -> C2286; JLC Price (none) -> 0.004; MPN (none) -> KT-0603R
- R?: renamed from R7; value ?220R? -> 51R; JLC Part Number (none) -> C23197; JLC Price (none) -> 0.0008; MPN (none) -> 0603WAF510JT5E
- R?: renamed from R4; JLC Part Number (none) -> C25804; JLC Price (none) -> 0.0007; MPN (none) -> 0603WAF1002T5E
- R?: renamed from R5; JLC Part Number (none) -> C21190; JLC Price (none) -> 0.0007; MPN (none) -> 0603WAF1001T5E
- R?: renamed from R10; value 4k7R -> 4.7kR; JLC Part Number (none) -> C23162; JLC Price (none) -> 0.0008; MPN (none) -> 0603WAF4701T5E
- R?: renamed from R1; footprint 0_Resistors:R_0402_1005_DensityHigh -> 0_Resistors:R_0603_1608_DensityHigh; JLC Part Number (none) -> C25190; JLC Price (none) -> 0.0008; MPN (none) -> 0603WAF270JT5E
- R?: renamed from R6; footprint 0_Resistors:R_0402_1005_DensityHigh -> 0_Resistors:R_0603_1608_DensityHigh; JLC Part Number (none) -> C21190; JLC Price (none) -> 0.0007; MPN (none) -> 0603WAF1001T5E
- R?: renamed from R2; footprint 0_Resistors:R_0402_1005_DensityHigh -> 0_Resistors:R_0603_1608_DensityHigh; JLC Part Number (none) -> C25190; JLC Price (none) -> 0.0008; MPN (none) -> 0603WAF270JT5E
- R?: renamed from R3; JLC Part Number (none) -> C25105; JLC Price (none) -> 0.0004; MPN (none) -> 0402WGF330JTCE
- R?: renamed from R8; value ?220R? -> 51R; JLC Part Number (none) -> C23197; JLC Price (none) -> 0.0008; MPN (none) -> 0603WAF510JT5E
- R?: renamed from R9; value 4k7R -> 4.7kR; JLC Part Number (none) -> C23162; JLC Price (none) -> 0.0008; MPN (none) -> 0603WAF4701T5E
- U? (x2): renamed from U1; value RP2350_80QFN -> RP2350B; Farnell Link (none) -> https://uk.farnell.com/raspberry-pi/rp2350b-tr7/mcu-32bit-1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; Farnell Part Number (none) -> N/A; Farnell Price (none) -> N/A; JLC Part Number (none) -> C42415655; JLC Price (none) -> 0.89; MPN (none) -> RP2350B
- U?: renamed from U2; Farnell Link (none) -> https://uk.farnell.com/infineon/s25fl128lagmfi013/flash-mem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; Farnell Part Number (none) -> 4128033; Farnell Price (none) -> 1.94; JLC Part Number (none) -> C97521; JLC Price (none) -> 1.13; Supplier Link https://uk.farnell.com/infineon/s25fl128lagmfi013/flash-mem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 -> (none)
- X?: renamed from X1; Farnell Link (none) -> https://uk.farnell.com/abracon/abm8-272-t3/crystal-12mhz-10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; Farnell Part Number (none) -> 4331750; Farnell Price (none) -> 0.67; JLC Part Number (none) -> C20625731; JLC Price (none) -> 0.25; MPN (none) -> ABM8-272-T3
Connections:
- net I2C_SCL: now also U?.21 (GPIO21)
- net I2C_SDA: now also U?.20 (GPIO20)
- net SD_CLK: now also U?.16 (GPIO16)
- net SD_CMD: now also U?.17 (GPIO17)
- net SD_DAT0: now also U?.14 (GPIO15)
- net SD_DAT1: now also U?.13 (GPIO14)
- net SD_DAT2: now also U?.19 (GPIO19)
- net SD_DAT3: now also U?.18 (GPIO18)
- net STATUS_BUZZER+: now also U?.45 (GPIO36)
- net STATUS_BUZZER-: now also U?.44 (GPIO35)
- net STATUS_LED_G: now also U?.48 (GPIO39)
- net STATUS_LED_R: now also U?.47 (GPIO38)
- net VBAT_sense: now also U?.58 (GPIO47_ADC7)
- net FIRE_SIGNAL: now reaches U?.1 (GPIO4)
- net PYRO_ST1: now reaches U?.11 (GPIO12)
- net PYRO_IN: now reaches U?.12 (GPIO13)
- net ARM_SIGNAL: now reaches U?.2 (GPIO5)
- net FILL_SIGNAL: now reaches U?.3 (GPIO6)
- net RJ45_LED2: now reaches U?.4 (GPIO7)
- net Servo3_PWM: now reaches U?.53 (GPIO42_ADC2)
- net Servo2_PWM: now reaches U?.55 (GPIO44_ADC4)
- net Servo1_PWM: now reaches U?.57 (GPIO46_ADC6)
- net RS485_TX: now reaches U?.6 (GPIO8)
- net RS485_RX: now reaches U?.7 (GPIO9)
- net RJ45_LED1: now reaches U?.8 (GPIO10)
- net PYRO_ST2: now reaches U?.9 (GPIO11)
- no-connect marks 9 -> 21
Other:
- note removed: "1v1 VDD Decoupling"
- note removed: "3v3 VDD Decoupling All 100nF"
- note removed: "4.7uF below VREG"
- note removed: "I2C Pull Ups"
- note removed: "Jumper to program with USB"
- company: (none) -> ${COMPANY}
- title: (none) -> MCU & Peripherals
- moved on the sheet: BUZ?, C?, D?, J?, L?, LED?, R?, U?, U?A, U?B, X?

Commit message: Example files update
Parts:
- gave numbers to parts that had none: 41

Commit message: Major sensor suite board changes, start of PCB layout
Parts:
- BUZ1: footprint 0_Passives:BUZZER,7.5x7.5mm -> 0_Passives:BUZZER,5x5mm
- J2, J402: now fitted
- R4: footprint 0_Resistors:R_0603_1608_DensityHigh -> 0_Resistors:R_0402_1005_DensityMedium
Connections:
- net ARM_SIGNAL is gone; now on net SD_DAT0: U1.2 (GPIO5)
- net FILL_SIGNAL is gone; now on net SD_CLK: U1.3 (GPIO6)
- net FIRE_SIGNAL is gone; now on net SD_DAT1: U1.1 (GPIO4)
- net RJ45_LED2 is gone; now on net SD_CMD: U1.4 (GPIO7)
- net RS485_RX is gone; now on net SD_DAT2: U1.7 (GPIO9)
- net RS485_TX is gone; now on net SD_DAT3: U1.6 (GPIO8)
- net SD_CLK: no longer U1.16 (GPIO16)
- net SD_CMD: no longer U1.17 (GPIO17)
- net SD_DAT0: no longer U1.14 (GPIO15)
- net SD_DAT1: no longer U1.13 (GPIO14)
- net SD_DAT2: no longer U1.19 (GPIO19)
- net SD_DAT3: no longer U1.18 (GPIO18)
- net PYRO_IN: no longer names the net of U1.12 (GPIO13)
- net PYRO_ST1: no longer names the net of U1.11 (GPIO12)
- net PYRO_ST2: no longer names the net of U1.9 (GPIO11)
- net RJ45_LED1: no longer names the net of U1.8 (GPIO10)
- net Servo1_PWM: no longer names the net of U1.57 (GPIO46_ADC6)
- net Servo2_PWM: no longer names the net of U1.55 (GPIO44_ADC4)
- net Servo3_PWM: no longer names the net of U1.53 (GPIO42_ADC2)
- no-connect marks 21 -> 28
Other:
- moved on the sheet: R10, R9

Commit message: Minor schematic adjustments
Parts:
- BUZ1: JLC Price 0.17 -> (none); JLC_MPN (none) -> MLT-7525; MPN MLT-7525 -> (none)
- C1, C15, C2, C3: JLC Price 0.0035 -> (none); JLC_MPN (none) -> CL05A475MP5NRNC; MPN CL05A475MP5NRNC -> GPC0402475; Package (none) -> C0402; Supplier (none) -> Generic
- C10, C11, C12, C13, C14, C4, C5, C6, C7, C8, C9: JLC Price 0.0009 -> (none); JLC_MPN (none) -> CL05B104KO5NNNC; MPN CL05B104KO5NNNC -> GPC0402104; Package (none) -> C0402; Supplier (none) -> Generic
- C16, C17: JLC Price 0.0007 -> (none); JLC_MPN (none) -> 0402CG150J500NT; MPN 0402CG150J500NT -> GPC0402150; Package (none) -> C0402; Supplier (none) -> Generic
- C18, C19: JLC Price 0.002 -> (none); JLC_MPN (none) -> CC0603KRX7R9BB104; MPN CC0603KRX7R9BB104 -> GPC0402104; Package (none) -> C0603; Supplier (none) -> Generic
- D1: JLC Price 0.0064 -> (none); Supplier (none) -> Farnell
- J1: Farnell Link https://uk.farnell.com/molex/47219-2001/connector-micro-sd-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 -> (none); Farnell Part Number 2614940 -> (none); Farnell Price 1.87 -> (none); JLC Price 0.43 -> (none); Order Code (none) -> 2614940; Supplier (none) -> Farnell; Supplier Link (none) -> https://uk.farnell.com/molex/47219-2001/connector-micro-sd-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
- J2, J402: JLC Price N/A -> (none); MPN N/A -> (none); Supplier (none) -> Farnell
- J401: Farnell Link https://uk.farnell.com/molex/502352-0201/wtb-conn-header-2p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 -> (none); Farnell Part Number 3103081 -> (none); Farnell Price 0.95 -> (none); JLC Price 0.22 -> (none); Order Code (none) -> 3103081; Supplier (none) -> Farnell; Supplier Link (none) -> https://uk.farnell.com/molex/502352-0201/wtb-conn-header-2p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
- L1: Farnell Link https://uk.farnell.com/abracon/aota-b201610s3r3-101-t/power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 -> (none); Farnell Part Number 4568814 -> (none); Farnell Price 1.4 -> (none); JLC Price 0.14 -> (none); Order Code (none) -> 4568814; Supplier (none) -> Farnell; Supplier Link (none) -> https://uk.farnell.com/abracon/aota-b201610s3r3-101-t/power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
- LED1: JLC Price 0.009 -> (none); JLC_MPN (none) -> KT-0603G; MPN KT-0603G -> (none); Package (none) -> D0603; Supplier (none) -> Farnell
- LED2: JLC Price 0.004 -> (none); JLC_MPN (none) -> KT-0603R; MPN KT-0603R -> (none); Package (none) -> D0603; Supplier (none) -> Farnell
- R1, R2: JLC Price 0.0008 -> (none); JLC_MPN (none) -> 0603WAF270JT5E; MPN 0603WAF270JT5E -> GPR060327R; Package (none) -> R0603; Supplier (none) -> Generic
- R10, R9: JLC Price 0.0008 -> (none); JLC_MPN (none) -> 0603WAF4701T5E; MPN 0603WAF4701T5E -> GPR06034K7; Package (none) -> R0603; Supplier (none) -> Generic
- R3: JLC Price 0.0004 -> (none); JLC_MPN (none) -> 0402WGF330JTCE; MPN 0402WGF330JTCE -> GPR040233R; Package (none) -> R0402; Supplier (none) -> Generic
- R4: JLC Price 0.0007 -> (none); JLC_MPN (none) -> 0603WAF1001T5E; MPN 0603WAF1001T5E -> GPR06031K; Package (none) -> R0402; Supplier (none) -> Generic
- R5: JLC Price 0.0007 -> (none); JLC_MPN (none) -> 0603WAF1002T5E; MPN 0603WAF1002T5E -> GPR060310K; Package (none) -> R0603; Supplier (none) -> Generic
- R6: JLC Price 0.0007 -> (none); JLC_MPN (none) -> 0603WAF1001T5E; MPN 0603WAF1001T5E -> GPR06031K; Package (none) -> R0603; Supplier (none) -> Generic
- R7, R8: JLC Price 0.0008 -> (none); JLC_MPN (none) -> 0603WAF510JT5E; MPN 0603WAF510JT5E -> GPR060351R; Package (none) -> R0603; Supplier (none) -> Generic
- U1: Farnell Link https://uk.farnell.com/raspberry-pi/rp2350b-tr7/mcu-32bit-1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 -> (none); Farnell Part Number N/A -> (none); Farnell Price N/A -> (none); JLC Price 0.89 -> (none); Package (none) -> QFN-80; Supplier (none) -> Farnell; Supplier Link (none) -> https://uk.farnell.com/raspberry-pi/rp2350b-tr7/mcu-32bit-1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
- U2: Farnell Link https://uk.farnell.com/infineon/s25fl128lagmfi013/flash-mem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 -> (none); Farnell Part Number 4128033 -> (none); Farnell Price 1.94 -> (none); JLC Price 1.13 -> (none); Order Code (none) -> 4128033; Package (none) -> SOIC-8; Supplier (none) -> Farnell; Supplier Link (none) -> https://uk.farnell.com/infineon/s25fl128lagmfi013/flash-mem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
- X1: Farnell Link https://uk.farnell.com/abracon/abm8-272-t3/crystal-12mhz-10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 -> (none); Farnell Part Number 4331750 -> (none); Farnell Price 0.67 -> (none); JLC Price 0.25 -> (none); Order Code (none) -> 4331750; Supplier (none) -> Farnell; Supplier Link (none) -> https://uk.farnell.com/abracon/abm8-272-t3/crystal-12mhz-10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
