File: CanSat_SensorSuite/SubSchematics/PosSensors.kicad_sch (KiCad schematic)
At the start: 2 parts, among them IC102 MS560702BA03-50

Commit message: Major sensor suite board changes, start of PCB layout
Parts:
- added C202: 100nF, 0_Capacitors:C_0603_1608_DensityHigh, symbol Sense&ControlBoard_symbol_library.pretty:C_0402
- added U202: LSM6DSOQTR, 0_Sensors:LSM6DSOQTR, symbol 0_Sensors:LSM6DSOQTR
- C201: renamed from C106; footprint Sense&ControlBoard_footprint_library:C_0402_1005Metric -> 0_Capacitors:C_0603_1608_DensityHigh
- U201: renamed from IC102; footprint MS5607-02BA03 -> 0_Sensors:MS5607-02BA03; MPN (none) -> MS560702BA03-50; Manufacturer_Name TE Connectivity -> (none); Manufacturer_Part_Number MS560702BA03-50 -> (none); Supplier (none) -> Farnell; Supplier Link (none) -> https://uk.farnell.com/sensor-solutions-te-connectivity/ms5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; Supplier Price (none) -> 7.88
Connections:
- net +3V3: now also C202.1, U202.12 (CS), U202.5 (VCCIO), U202.8 (VCC)
- net GND: now also C202.2, U202.1 (SA0), U202.2 (SDX), U202.3 (SCX), U202.6 (GND), U202.7 (GND)
- net I2C_SCL: now also U202.13 (SCL)
- net I2C_SDA: now also U202.14 (SDA)
- new net: U202.10 (NC), U202.11 (NC)
- no-connect marks 3 -> 5
Other:
- note added: "LSM6DSOQTR"
- note removed: "???"
- note removed: "Potential Baros: MS5607"
- note removed: "Potential IMUs: BNO055 - £7 JLC / £9 Mouser + High performance + Sensor fusion functionality - Not on Farnell"
- moved on the sheet: C201, U201

Commit message: Minor schematic adjustments
Parts:
- C201, C202: MPN (none) -> GPC0402104; Package (none) -> C0603; Supplier (none) -> Generic
- U201: Supplier Price 7.88 -> (none)
- U202: Supplier Price 2.36 -> (none)
Changed lines of the file:
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@@
 			)
 		)
-		(property "Description" ""
+		(property "Description" "SMD 0603 MLCC capacitor"
 			(at 149.86 199.39 0)
 			(effects
@@
 			)
 		)
-		(property "MPN" ""
+		(property "MPN" "GPC0402104"
 			(at 149.86 199.39 0)
 			(effects
@@
 			)
 		)
-		(property "Supplier" ""
+		(property "Supplier" "Generic"
+			(at 149.86 199.39 0)
+			(effects
+				(font
+					(size 1.27 1.27)
+				)
+				(hide yes)
+			)
+		)
+		(property "Package" "C0603"
 			(at 149.86 199.39 0)
 			(effects
@@
 			)
 		)
-		(property "Description" ""
+		(property "Description" "SMD 0603 MLCC capacitor"
 			(at 151.13 107.95 0)
 			(effects
@@
 			)
 		)
-		(property "MPN" ""
+		(property "MPN" "GPC0402104"
 			(at 151.13 107.95 0)
 			(effects
@@
 			)
 		)
-		(property "Supplier" ""
+		(property "Supplier" "Generic"
+			(at 151.13 107.95 0)
+			(effects
+				(font
+					(size 1.27 1.27)
+				)
+				(hide yes)
+			)
+		)
+		(property "Package" "C0603"
 			(at 151.13 107.95 0)
 			(effects
@@
 			)
 		)
-		(property "Supplier Price" "2.36"
-			(at 163.83 160.02 0)
-			(effects
-				(font
-					(size 1.27 1.27)
-				)
-				(hide yes)
-			)
-		)
 		(property "Supplier Link" "https://uk.farnell.com/stmicroelectronics/lsm6dsoqtr/inemo-inertial-module-3-6v-tri/dp/4209821"
 			(at 168.91 152.4 0)
+			(effects
+				(font
+					(size 1.27 1.27)
+				)
+				(hide yes)
+			)
+		)
+		(property "Package" ""
+			(at 166.37 101.6 0)
 			(effects
 				(font
@@
 			)
 		)
-		(property "Supplier Price" "7.88"
-			(at 162.56 195.58 0)
-			(effects
-				(font
-					(size 1.27 1.27)
-				)
-				(hide yes)
-			)
-		)
 		(property "Supplier Link" "https://uk.farnell.com/sensor-solutions-te-connectivity/ms560702ba03-50/sensor-barometric-0-01-1-2bar/dp/2362660"
 			(at 162.56 195.58 0)
 			(effects
+				(font
+					(size 1.27 1.27)
+				)
+				(hide yes)
+			)
+		)
+		(property "Package" ""
+			(at 162.56 195.58 0)
+			(effects
