File: CanSat_SensorSuite/SubSchematics/USBC_Battery Supply.kicad_sch (KiCad schematic)
At the start: 28 parts, among them J4 XT30_THT_H, J5 USBC_Conn, U4 NCP1117_3.3, U5 MIC29302AWD, U7 NCP1117_3.3

Commit message: Major sensor suite board changes, start of PCB layout
Parts:
- F1: renamed from F4; footprint 0_Passives:Fuse_2512_6332Metric -> 0_Power:Fuse_1210_3225Metric
- U5: footprint 0_Power:TO-252-5_TabPin3 -> 0_Power:MIC29302AWD
- renumbered C21 to C20, C20 to C21, C24 to C22, C25 to C23, C26 to C24, C27 to C25, D3 to D2, J5 to J3, LED6 to LED3, R22 to R11, R21 to R12, R20 to R13, R15 to R14, R16 to R15, R17 to R16, R13 to R17, U7 to U3
Changed lines of the file:
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@@
 	(rectangle
 		(start 102.87 44.45)
-		(end 316.23 125.73)
+		(end 316.23 121.92)
 		(stroke
 			(width 1)
@@
 	(text "Battery Voltage\nMonitoring"
 		(exclude_from_sim no)
-		(at 107.95 191.77 0)
+		(at 101.6 185.42 0)
 		(effects
 			(font
@@
 	(text "~0.45 Gain\n7.2V -> 3.3V"
 		(exclude_from_sim no)
-		(at 107.95 199.39 0)
+		(at 101.6 193.04 0)
 		(effects
 			(font
@@
 	(text_box "USB Data & Power"
 		(exclude_from_sim no)
-		(at 102.87 116.205 0)
+		(at 102.87 113.03 0)
 		(size 213.36 9.525)
 		(margins 1.9049 1.9049 1.9049 1.9049)
@@
 		(on_board yes)
 		(dnp no)
-		(property "Reference" "C21"
+		(property "Reference" "C20"
 			(at 233.045 74.93 90)
 			(effects
@@
 			(project "CanSat_SensorSuite"
 				(path "/0650c7a8-acba-429c-9f8e-eec0baf0bc1c/459e6a54-4354-4cbe-b679-1f9dcd1ee4fd/982efe7d-f5a1-469a-a12e-4fb13ad93078"
-					(reference "C21")
+					(reference "C20")
 					(unit 1)
 				)
@@
 			)
 		)
-		(property "Footprint" "0_Power:TO-252-5_TabPin3"
+		(property "Footprint" "0_Power:MIC29302AWD"
 			(at 219.71 233.68 0)
 			(effects
@@
 		(on_board yes)
 		(dnp no)
-		(property "Reference" "C25"
+		(property "Reference" "C23"
 			(at 256.794 163.83 90)
 			(effects
@@
 			(project "CanSat_SensorSuite"
 				(path "/0650c7a8-acba-429c-9f8e-eec0baf0bc1c/459e6a54-4354-4cbe-b679-1f9dcd1ee4fd/982efe7d-f5a1-469a-a12e-4fb13ad93078"
-					(reference "C25")
+					(reference "C23")
 					(unit 1)
 				)
@@
 		(on_board yes)
 		(dnp no)
-		(property "Reference" "J5"
+		(property "Reference" "J3"
 			(at 115.57 59.69 0)
 			(effects
@@
 			(project "CanSat_SensorSuite"
 				(path "/0650c7a8-acba-429c-9f8e-eec0baf0bc1c/459e6a54-4354-4cbe-b679-1f9dcd1ee4fd/982efe7d-f5a1-469a-a12e-4fb13ad93078"
-					(reference "J5")
+					(reference "J3")
 					(unit 1)
 				)
@@
 		(on_board yes)
 		(dnp no)
-		(property "Reference" "D3"
+		(property "Reference" "D2"
 			(at 176.276 86.868 0)
 			(effects
@@
 			(project "CanSat_SensorSuite"
 				(path "/0650c7a8-acba-429c-9f8e-eec0baf0bc1c/459e6a54-4354-4cbe-b679-1f9dcd1ee4fd/982efe7d-f5a1-469a-a12e-4fb13ad93078"
-					(reference "D3")
+					(reference "D2")
 					(unit 1)
 				)
@@
 		(on_board yes)
 		(dnp no)
-		(property "Reference" "U7"
+		(property "Reference" "U3"
 			(at 245.11 57.15 0)
 			(effects
@@
 			(project "CanSat_SensorSuite"
 				(path "/0650c7a8-acba-429c-9f8e-eec0baf0bc1c/459e6a54-4354-4cbe-b679-1f9dcd1ee4fd/982efe7d-f5a1-469a-a12e-4fb13ad93078"
-					(reference "U7")
+					(reference "U3")
 					(unit 1)
 				)
@@
 		(on_board yes)
 		(dnp no)
-		(property "Reference" "R17"
+		(property "Reference" "R16"
 			(at 257.81 217.17 90)
 			(effects
@@
 			(project "CanSat_SensorSuite"
 				(path "/0650c7a8-acba-429c-9f8e-eec0baf0bc1c/459e6a54-4354-4cbe-b679-1f9dcd1ee4fd/982efe7d-f5a1-469a-a12e-4fb13ad93078"
-					(reference "R17")
+					(reference "R16")
 					(unit 1)
 				)
@@
 		(on_board yes)
 		(dnp no)
-		(property "Reference" "R16"
+		(property "Reference" "R15"
 			(at 257.81 207.01 90)
 			(effects
@@
 			(project "CanSat_SensorSuite"
 				(path "/0650c7a8-acba-429c-9f8e-eec0baf0bc1c/459e6a54-4354-4cbe-b679-1f9dcd1ee4fd/982efe7d-f5a1-469a-a12e-4fb13ad93078"
-					(reference "R16")
+					(reference "R15")
 					(unit 1)
 				)
@@
 		(on_board yes)
 		(dnp no)
-		(property "Reference" "R20"
+		(property "Reference" "R13"
 			(at 276.77 85.16 90)
 			(effects
@@
 			(project "CanSat_SensorSuite"
 				(path "/0650c7a8-acba-429c-9f8e-eec0baf0bc1c/459e6a54-4354-4cbe-b679-1f9dcd1ee4fd/982efe7d-f5a1-469a-a12e-4fb13ad93078"
-					(reference "R20")
+					(reference "R13")
 					(unit 1)
 				)
@@
 		(on_board yes)
 		(dnp no)
-		(property "Reference" "R15"
+		(property "Reference" "R14"
 			(at 273.558 173.99 90)
 			(effects
@@
 			(project "CanSat_SensorSuite"
 				(path "/0650c7a8-acba-429c-9f8e-eec0baf0bc1c/459e6a54-4354-4cbe-b679-1f9dcd1ee4fd/982efe7d-f5a1-469a-a12e-4fb13ad93078"
-					(reference "R15")
+					(reference "R14")
 					(unit 1)
 				)
@@
 		(on_board yes)
 		(dnp no)
-		(property "Reference" "LED6"
+		(property "Reference" "LED3"
 			(at 276.59 77.58 90)
 			(effects
@@
 			(project "CanSat_SensorSuite"
 				(path "/0650c7a8-acba-429c-9f8e-eec0baf0bc1c/459e6a54-4354-4cbe-b679-1f9dcd1ee4fd/982efe7d-f5a1-469a-a12e-4fb13ad93078"
-					(reference "LED6")
+					(reference "LED3")
 					(unit 1)
 				)
@@
 		(on_board yes)
 		(dnp no)
-		(property "Reference" "R22"
+		(property "Reference" "R11"
 			(at 149.225 100.33 90)
 			(effects
@@
 			(project "CanSat_SensorSuite"
 				(path "/0650c7a8-acba-429c-9f8e-eec0baf0bc1c/459e6a54-4354-4cbe-b679-1f9dcd1ee4fd/982efe7d-f5a1-469a-a12e-4fb13ad93078"
-					(reference "R22")
+					(reference "R11")
 					(unit 1)
 				)
@@
 		(on_board yes)
 		(dnp no)
-		(property "Reference" "R21"
+		(property "Reference" "R12"
 			(at 158.75 100.33 90)
 			(effects
@@
 			(project "CanSat_SensorSuite"
 				(path "/0650c7a8-acba-429c-9f8e-eec0baf0bc1c/459e6a54-4354-4cbe-b679-1f9dcd1ee4fd/982efe7d-f5a1-469a-a12e-4fb13ad93078"
-					(reference "R21")
+					(reference "R12")
 					(unit 1)
 				)
@@
 		(on_board yes)
 		(dnp no)
-		(property "Reference" "F4"
+		(property "Reference" "F1"
 			(at 158.75 65.278 0)
 			(effects
@@
 			)
 		)
-		(property "Footprint" "0_Passives:Fuse_2512_6332Metric"
+		(property "Footprint" "0_Power:Fuse_1210_3225Metric"
 			(at 164.338 67.31 90)
 			(effects
@@
 			(project "CanSat_SensorSuite"
 				(path "/0650c7a8-acba-429c-9f8e-eec0baf0bc1c/459e6a54-4354-4cbe-b679-1f9dcd1ee4fd/982efe7d-f5a1-469a-a12e-4fb13ad93078"
-					(reference "F4")
+					(reference "F1")
 					(unit 1)
 				)
@@
 		(on_board yes)
 		(dnp no)
-		(property "Reference" "C27"
+		(property "Reference" "C25"
 			(at 299.72 217.17 90)
 			(effects
@@
 			(project "CanSat_SensorSuite"
 				(path "/0650c7a8-acba-429c-9f8e-eec0baf0bc1c/459e6a54-4354-4cbe-b679-1f9dcd1ee4fd/982efe7d-f5a1-469a-a12e-4fb13ad93078"
-					(reference "C27")
+					(reference "C25")
 					(unit 1)
 				)
@@
 		(on_board yes)
 		(dnp no)
-		(property "Reference" "R13"
+		(property "Reference" "R17"
 			(at 271.018 217.17 90)
 			(effects
@@
 			(project "CanSat_SensorSuite"
 				(path "/0650c7a8-acba-429c-9f8e-eec0baf0bc1c/459e6a54-4354-4cbe-b679-1f9dcd1ee4fd/982efe7d-f5a1-469a-a12e-4fb13ad93078"
-					(reference "R13")
+					(reference "R17")
 					(unit 1)
 				)
@@
 		(on_board yes)
 		(dnp no)
-		(property "Reference" "C20"
+		(property "Reference" "C21"
 			(at 257.175 74.93 90)
 			(effects
@@
 			(project "CanSat_SensorSuite"
 				(path "/0650c7a8-acba-429c-9f8e-eec0baf0bc1c/459e6a54-4354-4cbe-b679-1f9dcd1ee4fd/982efe7d-f5a1-469a-a12e-4fb13ad93078"
-					(reference "C20")
+					(reference "C21")
 					(unit 1)
 				)
@@
 		(on_board yes)
 		(dnp no)
-		(property "Reference" "C26"
+		(property "Reference" "C24"
 			(at 287.02 217.17 90)
 			(effects
@@
 			(project "CanSat_SensorSuite"
 				(path "/0650c7a8-acba-429c-9f8e-eec0baf0bc1c/459e6a54-4354-4cbe-b679-1f9dcd1ee4fd/982efe7d-f5a1-469a-a12e-4fb13ad93078"
-					(reference "C26")
+					(reference "C24")
 					(unit 1)
 				)
@@
 		(on_board yes)
 		(dnp no)
-		(property "Reference" "C24"
+		(property "Reference" "C22"
 			(at 217.17 163.83 90)
 			(effects
@@
 			(project "CanSat_SensorSuite"
 				(path "/0650c7a8-acba-429c-9f8e-eec0baf0bc1c/459e6a54-4354-4cbe-b679-1f9dcd1ee4fd/982efe7d-f5a1-469a-a12e-4fb13ad93078"
-					(reference "C24")
+					(reference "C22")
 					(unit 1)
 				)

Commit message: Minor schematic adjustments
Parts:
- C20, C21: MPN (none) -> GPC0402103; Package (none) -> C0603; Supplier (none) -> Generic
- C22, C23: JLC Part Number (none) -> C57112; JLC_PART C57112 -> (none); MPN (none) -> GPC0402103; Package (none) -> C0603; Supplier (none) -> Generic
- C24, C25: JLC Part Number (none) -> C19702; JLC_PART C19702 -> (none); MPN (none) -> GPC0603106; Package (none) -> C0603; Supplier (none) -> Generic
- D2, F1, J3: Supplier (none) -> Farnell
- F2, F3: JLC Part Number (none) -> C634245; JLC_PART C634245 -> (none); Supplier (none) -> Farnell
- J4: JLC Part Number (none) -> C431092; JLC_PART C431092 -> (none); Manufacturer_Name Multicomp Pro -> (none); Supplier (none) -> Farnell
- LED3: JLC Price 0.004 -> (none); JLC_MPN (none) -> KT-0603R; MPN KT-0603R -> (none); Package (none) -> D0603; Supplier (none) -> Farnell
- LED4, LED5: JLC Part Number (none) -> C2286; JLC_PART C2286 -> (none); Package (none) -> D0603; Supplier (none) -> Farnell
- R11, R12: MPN (none) -> GPR06035K1; Package (none) -> R0603; Supplier (none) -> Generic
- R13: JLC Price 0.0008 -> (none); JLC_MPN (none) -> 0603WAF510JT5E; MPN 0603WAF510JT5E -> GPR060351R; Package (none) -> R0603; Supplier (none) -> Generic
- R14, R17: JLC Part Number (none) -> C23197; JLC_PART C23197 -> (none); MPN (none) -> GPR060351R; Package (none) -> R0603; Supplier (none) -> Generic
- R15: JLC Part Number (none) -> C23179; JLC_PART C23179 -> (none); Package (none) -> R0603; Supplier (none) -> Generic
- R16: JLC Part Number (none) -> C22787; JLC_PART C22787 -> (none); Package (none) -> R0603; Supplier (none) -> Generic
- R18: JLC Part Number (none) -> C23178; JLC_PART C23178 -> (none); MPN (none) -> GPR0402470K; Package (none) -> R0603; Supplier (none) -> Generic
- R19: JLC Part Number (none) -> C23150; JLC_PART C23150 -> (none); MPN (none) -> GPR0402390K; Package (none) -> R0603; Supplier (none) -> Generic
- S1: JLC Part Number (none) -> C17179519; JLC_PART C17179519 -> (none); Supplier (none) -> Farnell
- U3: Package (none) -> SOT-223-3; Supplier (none) -> Farnell
- U4: JLC Part Number (none) -> C146799; JLC_PART C146799 -> (none); Package (none) -> SOT-223-3; Supplier (none) -> Farnell
- U5: JLC Part Number (none) -> C627907; JLC_PART C627907 -> (none); Supplier (none) -> Farnell; Supplier Link (none) -> https://uk.farnell.com/microchip/mic29302awd-tr/ldo-adj-1-2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; Supplier_Link https://uk.farnell.com/microchip/mic29302awd-tr/ldo-adj-1-2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 -> (none)
