File: SensorSuite_Circular/TopBoard_Control/TopBoard_Control.kicad_pcb (KiCad board)
At the start: 4 copper layers, 50 x 110 mm, 88 parts, among them J1 Micro_SD_Card, J101 SPS30, J104 JST-S5B-ZR, J2 Pin_01x02, J3 USBC_Conn, J4 XT30_THT_H, J401 Molex_01x02, J402 Conn_02x03, U1 RP2350B, U102 ZMOD4410AI1R, U103 STC31-C-R3, U2 S25FL128, U201 MS560702BA03-50, U202 LSM6DSOQTR, U3 NCP1117_3.3, U4 NCP1117_3.3, U5 MIC29302AWD, X1 ABM8-272-T3

Commit message: upload moxon matlab
Parts:
- moved FID301 9.12 mm to (125.3, 133.1)
- moved BUZ1 9.12 mm to (166.0, 97.8)
- moved C1 9.12 mm to (145.2, 80.0)
- moved C10 9.12 mm to (148.3, 80.1)
- moved C101 9.12 mm to (161.8, 120.2)
- moved C102 9.12 mm to (156.1, 121.5)
- moved C103 9.12 mm to (139.1, 121.9)
- moved C11 9.12 mm to (138.5, 83.0)
- moved C12 9.12 mm to (138.9, 86.9)
- moved C13 9.12 mm to (139.6, 94.7)
- moved C14 9.12 mm to (152.8, 93.3)
- moved C15 9.12 mm to (151.3, 82.5)
- moved C16 9.12 mm to (152.3, 96.9)
- moved C17 9.12 mm to (154.3, 94.9)
- moved C18 9.12 mm to (132.0, 84.4)
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